File: poc_controller/poc_controller_sensors.sch (KiCad schematic (older format))
At the start: 10 parts

Commit message: Start assigning footprints and cleaning things up.
Parts:
- gave numbers to parts that had none: 10
Changed lines of the file:
@@
 $Descr A4 11693 8268
 encoding utf-8
-Sheet 2 3
+Sheet 2 4
 Title ""
 Date ""
@@
 $EndDescr
 $Comp
-L LSM6DS3H U?
+L LSM6DS3H U5
 U 1 1 5A01288C
 P 7350 2650
-F 0 "U?" H 7750 2650 60  0000 C CNN
+F 0 "U5" H 7750 2650 60  0000 C CNN
 F 1 "LSM6DS3H" H 7350 2650 60  0000 C CNN
 F 2 "" H 7350 2650 60  0001 C CNN
@@
 $EndComp
 $Comp
-L GND #PWR?
+L GND #PWR28
 U 1 1 5A01298A
 P 6700 3500
-F 0 "#PWR?" H 6700 3250 50  0001 C CNN
+F 0 "#PWR28" H 6700 3250 50  0001 C CNN
 F 1 "GND" H 6700 3350 50  0000 C CNN
 F 2 "" H 6700 3500 50  0001 C CNN
@@
 Connection ~ 6700 3400
 $Comp
-L +3.3V #PWR?
+L +3.3V #PWR25
 U 1 1 5A0129F8
 P 6200 3200
-F 0 "#PWR?" H 6200 3050 50  0001 C CNN
+F 0 "#PWR25" H 6200 3050 50  0001 C CNN
 F 1 "+3.3V" H 6200 3340 50  0000 C CNN
 F 2 "" H 6200 3200 50  0001 C CNN
@@
 $EndComp
 $Comp
-L CP1 C?
+L CP1 C11
 U 1 1 5A012A11
 P 6200 3350
-F 0 "C?" H 6225 3450 50  0000 L CNN
+F 0 "C11" H 6225 3450 50  0000 L CNN
 F 1 "100nF" H 6225 3250 50  0000 L CNN
 F 2 "" H 6200 3350 50  0001 C CNN
@@
 $EndComp
 $Comp
-L GND #PWR?
+L GND #PWR26
 U 1 1 5A012A42
 P 6200 3500
-F 0 "#PWR?" H 6200 3250 50  0001 C CNN
+F 0 "#PWR26" H 6200 3250 50  0001 C CNN
 F 1 "GND" H 6200 3350 50  0000 C CNN
 F 2 "" H 6200 3500 50  0001 C CNN
@@
 NoConn ~ 7950 3100
 $Comp
-L +3.3V #PWR?
+L +3.3V #PWR29
 U 1 1 5A012FB2
 P 8300 2700
-F 0 "#PWR?" H 8300 2550 50  0001 C CNN
+F 0 "#PWR29" H 8300 2550 50  0001 C CNN
 F 1 "+3.3V" H 8300 2840 50  0000 C CNN
 F 2 "" H 8300 2700 50  0001 C CNN
@@
 $EndComp
 $Comp
-L CP1 C?
+L CP1 C12
 U 1 1 5A012FCC
 P 8300 2850
-F 0 "C?" H 8325 2950 50  0000 L CNN
+F 0 "C12" H 8325 2950 50  0000 L CNN
 F 1 "100nF" H 8325 2750 50  0000 L CNN
 F 2 "" H 8300 2850 50  0001 C CNN
@@
 $EndComp
 $Comp
-L GND #PWR?
+L GND #PWR30
 U 1 1 5A012FF1
 P 8300 3000
-F 0 "#PWR?" H 8300 2750 50  0001 C CNN
+F 0 "#PWR30" H 8300 2750 50  0001 C CNN
 F 1 "GND" H 8300 2850 50  0000 C CNN
 F 2 "" H 8300 3000 50  0001 C CNN
@@
 NoConn ~ 7950 2900
 $Comp
-L GND #PWR?
+L GND #PWR27
 U 1 1 5A0130C5
 P 6500 2600
-F 0 "#PWR?" H 6500 2350 50  0001 C CNN
+F 0 "#PWR27" H 6500 2350 50  0001 C CNN
 F 1 "GND" H 6500 2450 50  0000 C CNN
 F 2 "" H 6500 2600 50  0001 C CNN
@@
 	1200 1450 1500 1450
 $Comp
-L R R?
+L R R6
 U 1 1 5A013CB5
 P 8100 3000
-F 0 "R?" V 8180 3000 50  0000 C CNN
+F 0 "R6" V 8180 3000 50  0000 C CNN
 F 1 "4.7k" V 8100 3000 50  0000 C CNN
 F 2 "" V 8030 3000 50  0001 C CNN
@@
 	8100 2700 8100 2850
 $Comp
-L MAG3110 U?
+L MAG3110 U4
 U 1 1 5A014ADE
 P 3750 3700
-F 0 "U?" H 4150 3700 60  0000 C CNN
+F 0 "U4" H 4150 3700 60  0000 C CNN
 F 1 "MAG3110" H 3750 3700 60  0000 C CNN
 F 2 "" H 3750 3700 60  0001 C CNN
@@
 EXT_INT_2
 $Comp
-L GND #PWR?
+L GND #PWR22
 U 1 1 5A014C7A
 P 4800 3450
-F 0 "#PWR?" H 4800 3200 50  0001 C CNN
+F 0 "#PWR22" H 4800 3200 50  0001 C CNN
 F 1 "GND" H 4800 3300 50  0000 C CNN
 F 2 "" H 4800 3450 50  0001 C CNN
@@
 SDA
 $Comp
-L +3.3V #PWR?
+L +3.3V #PWR23
 U 1 1 5A014D65
 P 5000 4050
-F 0 "#PWR?" H 5000 3900 50  0001 C CNN
+F 0 "#PWR23" H 5000 3900 50  0001 C CNN
 F 1 "+3.3V" H 5000 4190 50  0000 C CNN
 F 2 "" H 5000 4050 50  0001 C CNN
@@
 $EndComp
 $Comp
-L CP1 C?
+L CP1 C10
 U 1 1 5A014DA9
 P 5000 4200
-F 0 "C?" H 5025 4300 50  0000 L CNN
+F 0 "C10" H 5025 4300 50  0000 L CNN
 F 1 "CP1" H 5025 4100 50  0000 L CNN
 F 2 "" H 5000 4200 50  0001 C CNN
@@
 Connection ~ 5000 4050
 $Comp
-L GND #PWR?
+L GND #PWR24
 U 1 1 5A014DEF
 P 5000 4350
-F 0 "#PWR?" H 5000 4100 50  0001 C CNN
+F 0 "#PWR24" H 5000 4100 50  0001 C CNN
 F 1 "GND" H 5000 4200 50  0000 C CNN
 F 2 "" H 5000 4350 50  0001 C CNN
@@
 	4350 4050 5000 4050
 $Comp
-L GND #PWR?
+L GND #PWR21
 U 1 1 5A014E63
 P 3050 4400
-F 0 "#PWR?" H 3050 4150 50  0001 C CNN
+F 0 "#PWR21" H 3050 4150 50  0001 C CNN
 F 1 "GND" H 3050 4250 50  0000 C CNN
 F 2 "" H 3050 4400 50  0001 C CNN
@@
 	3050 4250 3050 4400
 $Comp
-L CP1 C?
+L CP1 C9
 U 1 1 5A014F15
 P 2700 4300
-F 0 "C?" H 2725 4400 50  0000 L CNN
+F 0 "C9" H 2725 4400 50  0000 L CNN
 F 1 "100nF" H 2725 4200 50  0000 L CNN
 F 2 "" H 2700 4300 50  0001 C CNN
@@
 $EndComp
 $Comp
-L GND #PWR?
+L GND #PWR20
 U 1 1 5A014F44
 P 2700 4450
-F 0 "#PWR?" H 2700 4200 50  0001 C CNN
+F 0 "#PWR20" H 2700 4200 50  0001 C CNN
 F 1 "GND" H 2700 4300 50  0000 C CNN
 F 2 "" H 2700 4450 50  0001 C CNN
@@
 	2700 4150 3200 4150
 $Comp
-L +3.3V #PWR?
+L +3.3V #PWR18
 U 1 1 5A015071
 P 2200 3950
-F 0 "#PWR?" H 2200 3800 50  0001 C CNN
+F 0 "#PWR18" H 2200 3800 50  0001 C CNN
 F 1 "+3.3V" H 2200 4090 50  0000 C CNN
 F 2 "" H 2200 3950 50  0001 C CNN
@@
 $EndComp
 $Comp
-L CP1 C?
+L CP1 C7
 U 1 1 5A01509A
 P 2050 4200
-F 0 "C?" H 2075 4300 50  0000 L CNN
+F 0 "C7" H 2075 4300 50  0000 L CNN
 F 1 "1uF" H 2075 4100 50  0000 L CNN
 F 2 "" H 2050 4200 50  0001 C CNN
@@
 $EndComp
 $Comp
-L CP1 C?
+L CP1 C8
 U 1 1 5A0150D2
 P 2300 4200
-F 0 "C?" H 2325 4300 50  0000 L CNN
+F 0 "C8" H 2325 4300 50  0000 L CNN
 F 1 "100nF" H 2325 4100 50  0000 L CNN
 F 2 "" H 2300 4200 50  0001 C CNN
@@
 $EndComp
 $Comp
-L GND #PWR?
+L GND #PWR19
 U 1 1 5A015106
 P 2200 4450
-F 0 "#PWR?" H 2200 4200 50  0001 C CNN
+F 0 "#PWR19" H 2200 4200 50  0001 C CNN
 F 1 "GND" H 2200 4300 50  0000 C CNN
 F 2 "" H 2200 4450 50  0001 C CNN
@@
 	2200 3950 3200 3950
 $Comp
-L CP1 C?
+L CP1 C6
 U 1 1 5A01544B
 P 1650 3900
-F 0 "C?" H 1675 4000 50  0000 L CNN
+F 0 "C6" H 1675 4000 50  0000 L CNN
 F 1 "100nF" H 1675 3800 50  0000 L CNN
 F 2 "" H 1650 3900 50  0001 C CNN
@@
 $EndComp
 $Comp
-L GND #PWR?
+L GND #PWR17
 U 1 1 5A015490
 P 1650 4050
-F 0 "#PWR?" H 1650 3800 50  0001 C CNN
+F 0 "#PWR17" H 1650 3800 50  0001 C CNN
 F 1 "GND" H 1650 3900 50  0000 C CNN
 F 2 "" H 1650 4050 50  0001 C CNN

Commit message: More footprint assignment.
Parts:
- removed C10: CP1, symbol CP1
- removed C11, C12, C6, C8, C9: 100nF, symbol CP1
- removed C7: 1uF, symbol CP1
- added C10, C12, C6, C8, C9: 0.1uF, Capacitors_SMD:C_1206_HandSoldering, symbol C
- added C11: 0.1uF, Housings_LGA:Bosch_LGA-14_3x2.5mm_Pitch0.5mm, symbol C
- added C7: 1uF, Capacitors_SMD:C_1206_HandSoldering, symbol C
- R6: footprint (none) -> Resistors_SMD:R_1206_HandSoldering; Part Number (none) -> 311-4.70KMCT-ND
- U4: footprint (none) -> Housings_DFN_QFN:DFN-10_2x2mm_Pitch0.4mm; Part Number (none) -> MAG3110FCR1CT-ND
- U5: footprint (none) -> Housings_LGA:Bosch_LGA-14_3x2.5mm_Pitch0.5mm; Part Number (none) -> 497-16367-1-ND
Connections:
- net +3V3: now also C10.1, C11.1, C12.1, C7.1, C8.1
- net GND: now also C10.2, C11.2, C12.2, C6.2, C7.2, C8.2, C9.2
- net at U4.1 (Cap-A): now also C6.1
- net at U4.4 (Cap-R): now also C9.1
Changed lines of the file:
@@
 F 0 "U5" H 7750 2650 60  0000 C CNN
 F 1 "LSM6DS3H" H 7350 2650 60  0000 C CNN
-F 2 "" H 7350 2650 60  0001 C CNN
+F 2 "Housings_LGA:Bosch_LGA-14_3x2.5mm_Pitch0.5mm" H 7350 2650 60  0001 C CNN
 F 3 "" H 7350 2650 60  0001 C CNN
+F 4 "497-16367-1-ND" H 7350 2650 60  0001 C CNN "Part Number"
 	1    7350 2650
 	1    0    0    -1
@@
 $EndComp
 $Comp
-L CP1 C11
-U 1 1 5A012A11
-P 6200 3350
-F 0 "C11" H 6225 3450 50  0000 L CNN
-F 1 "100nF" H 6225 3250 50  0000 L CNN
-F 2 "" H 6200 3350 50  0001 C CNN
-F 3 "" H 6200 3350 50  0001 C CNN
-	1    6200 3350
-	1    0    0    -1
-$EndComp
-$Comp
 L GND #PWR26
 U 1 1 5A012A42
@@
 F 3 "" H 8300 2700 50  0001 C CNN
 	1    8300 2700
-	1    0    0    -1
-$EndComp
-$Comp
-L CP1 C12
-U 1 1 5A012FCC
-P 8300 2850
-F 0 "C12" H 8325 2950 50  0000 L CNN
-F 1 "100nF" H 8325 2750 50  0000 L CNN
-F 2 "" H 8300 2850 50  0001 C CNN
-F 3 "" H 8300 2850 50  0001 C CNN
-	1    8300 2850
 	1    0    0    -1
 $EndComp
@@
 F 0 "R6" V 8180 3000 50  0000 C CNN
 F 1 "4.7k" V 8100 3000 50  0000 C CNN
-F 2 "" V 8030 3000 50  0001 C CNN
+F 2 "Resistors_SMD:R_1206_HandSoldering" V 8030 3000 50  0001 C CNN
 F 3 "" H 8100 3000 50  0001 C CNN
+F 4 "311-4.70KMCT-ND" V 8100 3000 60  0001 C CNN "Part Number"
 	1    8100 3000
 	1    0    0    -1
@@
 F 0 "U4" H 4150 3700 60  0000 C CNN
 F 1 "MAG3110" H 3750 3700 60  0000 C CNN
-F 2 "" H 3750 3700 60  0001 C CNN
+F 2 "Housings_DFN_QFN:DFN-10_2x2mm_Pitch0.4mm" H 3750 3700 60  0001 C CNN
 F 3 "" H 3750 3700 60  0001 C CNN
+F 4 "MAG3110FCR1CT-ND" H 3750 3700 60  0001 C CNN "Part Number"
 	1    3750 3700
 	1    0    0    -1
@@
 	1    0    0    -1
 $EndComp
-$Comp
-L CP1 C10
-U 1 1 5A014DA9
-P 5000 4200
-F 0 "C10" H 5025 4300 50  0000 L CNN
-F 1 "CP1" H 5025 4100 50  0000 L CNN
-F 2 "" H 5000 4200 50  0001 C CNN
-F 3 "" H 5000 4200 50  0001 C CNN
-	1    5000 4200
-	1    0    0    -1
-$EndComp
 Connection ~ 5000 4050
 $Comp
@@
 	3050 4250 3050 4400
 $Comp
-L CP1 C9
-U 1 1 5A014F15
-P 2700 4300
-F 0 "C9" H 2725 4400 50  0000 L CNN
-F 1 "100nF" H 2725 4200 50  0000 L CNN
-F 2 "" H 2700 4300 50  0001 C CNN
-F 3 "" H 2700 4300 50  0001 C CNN
-	1    2700 4300
-	1    0    0    -1
-$EndComp
-$Comp
 L GND #PWR20
 U 1 1 5A014F44
@@
 $EndComp
 $Comp
-L CP1 C7
-U 1 1 5A01509A
-P 2050 4200
-F 0 "C7" H 2075 4300 50  0000 L CNN
-F 1 "1uF" H 2075 4100 50  0000 L CNN
-F 2 "" H 2050 4200 50  0001 C CNN
-F 3 "" H 2050 4200 50  0001 C CNN
-	1    2050 4200
-	1    0    0    -1
-$EndComp
-$Comp
-L CP1 C8
-U 1 1 5A0150D2
-P 2300 4200
-F 0 "C8" H 2325 4300 50  0000 L CNN
-F 1 "100nF" H 2325 4100 50  0000 L CNN
-F 2 "" H 2300 4200 50  0001 C CNN
-F 3 "" H 2300 4200 50  0001 C CNN
-	1    2300 4200
-	1    0    0    -1
-$EndComp
-$Comp
 L GND #PWR19
 U 1 1 5A015106
@@
 	2200 3950 3200 3950
 $Comp
-L CP1 C6
-U 1 1 5A01544B
-P 1650 3900
-F 0 "C6" H 1675 4000 50  0000 L CNN
-F 1 "100nF" H 1675 3800 50  0000 L CNN
-F 2 "" H 1650 3900 50  0001 C CNN
-F 3 "" H 1650 3900 50  0001 C CNN
-	1    1650 3900
-	1    0    0    -1
-$EndComp
-$Comp
 L GND #PWR17
 U 1 1 5A015490
@@
 Wire Wire Line
 	2900 3850 3200 3850
+$Comp
+L C C6
+U 1 1 5AB7EC4F
+P 1650 3900
+F 0 "C6" H 1675 4000 50  0000 L CNN
+F 1 "0.1uF" H 1675 3800 50  0000 L CNN
+F 2 "Capacitors_SMD:C_1206_HandSoldering" H 1688 3750 50  0001 C CNN
+F 3 "" H 1650 3900 50  0001 C CNN
+F 4 "311-1179-1-ND" H 1650 3900 60  0001 C CNN "Part Number"
+	1    1650 3900
+	1    0    0    -1
+$EndComp
+$Comp
+L C C8
+U 1 1 5AB7EE7A
+P 2300 4200
+F 0 "C8" H 2325 4300 50  0000 L CNN
+F 1 "0.1uF" H 2325 4100 50  0000 L CNN
+F 2 "Capacitors_SMD:C_1206_HandSoldering" H 2338 4050 50  0001 C CNN
+F 3 "" H 2300 4200 50  0001 C CNN
+F 4 "311-1179-1-ND" H 2300 4200 60  0001 C CNN "Part Number"
+	1    2300 4200
+	1    0    0    -1
+$EndComp
+$Comp
+L C C9
+U 1 1 5AB7EF1C
+P 2700 4300
+F 0 "C9" H 2725 4400 50  0000 L CNN
+F 1 "0.1uF" H 2725 4200 50  0000 L CNN
+F 2 "Capacitors_SMD:C_1206_HandSoldering" H 2738 4150 50  0001 C CNN
+F 3 "" H 2700 4300 50  0001 C CNN
+F 4 "311-1179-1-ND" H 2700 4300 60  0001 C CNN "Part Number"
+	1    2700 4300
+	1    0    0    -1
+$EndComp
+$Comp
+L C C10
+U 1 1 5AB7EFA4
+P 5000 4200
+F 0 "C10" H 5025 4300 50  0000 L CNN
+F 1 "0.1uF" H 5025 4100 50  0000 L CNN
+F 2 "Capacitors_SMD:C_1206_HandSoldering" H 5038 4050 50  0001 C CNN
+F 3 "" H 5000 4200 50  0001 C CNN
+F 4 "311-1179-1-ND" H 5000 4200 60  0001 C CNN "Part Number"
+	1    5000 4200
+	1    0    0    -1
+$EndComp
+$Comp
+L C C7
+U 1 1 5AB7F05A
+P 2050 4200
+F 0 "C7" H 2075 4300 50  0000 L CNN
+F 1 "1uF" H 2075 4100 50  0000 L CNN
+F 2 "Capacitors_SMD:C_1206_HandSoldering" H 2088 4050 50  0001 C CNN
+F 3 "" H 2050 4200 50  0001 C CNN
+F 4 "311-1356-1-ND" H 2050 4200 60  0001 C CNN "Part Number"
+	1    2050 4200
+	1    0    0    -1
+$EndComp
+$Comp
+L C C11
+U 1 1 5AB7F32E
+P 6200 3350
+F 0 "C11" H 6225 3450 50  0000 L CNN
+F 1 "0.1uF" H 6225 3250 50  0000 L CNN
+F 2 "Housings_LGA:Bosch_LGA-14_3x2.5mm_Pitch0.5mm" H 6238 3200 50  0001 C CNN
+F 3 "" H 6200 3350 50  0001 C CNN
+F 4 "311-1179-1-ND" H 6200 3350 60  0001 C CNN "Part Number"
+	1    6200 3350
+	1    0    0    -1
+$EndComp
+$Comp
+L C C12
+U 1 1 5AB7F374
+P 8300 2850
+F 0 "C12" H 8325 2950 50  0000 L CNN
+F 1 "0.1uF" H 8325 2750 50  0000 L CNN
+F 2 "Capacitors_SMD:C_1206_HandSoldering" H 8338 2700 50  0001 C CNN
+F 3 "" H 8300 2850 50  0001 C CNN
+F 4 "311-1179-1-ND" H 8300 2850 60  0001 C CNN "Part Number"
+	1    8300 2850
+	1    0    0    -1
+$EndComp
 $EndSCHEMATC

Commit message: More design and component selection.
Parts:
- renumbered U4 to U2, U5 to U3
Changed lines of the file:
@@
 LIBS:valves
 LIBS:quadcopter_lib
+LIBS:switches
 LIBS:poc_controller-cache
 EELAYER 25 0
@@
 $EndDescr
 $Comp
-L LSM6DS3H U5
+L LSM6DS3H U3
 U 1 1 5A01288C
 P 7350 2650
-F 0 "U5" H 7750 2650 60  0000 C CNN
+F 0 "U3" H 7750 2650 60  0000 C CNN
 F 1 "LSM6DS3H" H 7350 2650 60  0000 C CNN
 F 2 "Housings_LGA:Bosch_LGA-14_3x2.5mm_Pitch0.5mm" H 7350 2650 60  0001 C CNN
@@
 $EndComp
 $Comp
-L GND #PWR28
+L GND #PWR24
 U 1 1 5A01298A
 P 6700 3500
-F 0 "#PWR28" H 6700 3250 50  0001 C CNN
+F 0 "#PWR24" H 6700 3250 50  0001 C CNN
 F 1 "GND" H 6700 3350 50  0000 C CNN
 F 2 "" H 6700 3500 50  0001 C CNN
@@
 Connection ~ 6700 3400
 $Comp
-L +3.3V #PWR25
+L +3.3V #PWR21
 U 1 1 5A0129F8
 P 6200 3200
-F 0 "#PWR25" H 6200 3050 50  0001 C CNN
+F 0 "#PWR21" H 6200 3050 50  0001 C CNN
 F 1 "+3.3V" H 6200 3340 50  0000 C CNN
 F 2 "" H 6200 3200 50  0001 C CNN
@@
 $EndComp
 $Comp
-L GND #PWR26
+L GND #PWR22
 U 1 1 5A012A42
 P 6200 3500
-F 0 "#PWR26" H 6200 3250 50  0001 C CNN
+F 0 "#PWR22" H 6200 3250 50  0001 C CNN
 F 1 "GND" H 6200 3350 50  0000 C CNN
 F 2 "" H 6200 3500 50  0001 C CNN
@@
 NoConn ~ 7950 3100
 $Comp
-L +3.3V #PWR29
+L +3.3V #PWR25
 U 1 1 5A012FB2
 P 8300 2700
-F 0 "#PWR29" H 8300 2550 50  0001 C CNN
+F 0 "#PWR25" H 8300 2550 50  0001 C CNN
 F 1 "+3.3V" H 8300 2840 50  0000 C CNN
 F 2 "" H 8300 2700 50  0001 C CNN
@@
 $EndComp
 $Comp
-L GND #PWR30
+L GND #PWR26
 U 1 1 5A012FF1
 P 8300 3000
-F 0 "#PWR30" H 8300 2750 50  0001 C CNN
+F 0 "#PWR26" H 8300 2750 50  0001 C CNN
 F 1 "GND" H 8300 2850 50  0000 C CNN
 F 2 "" H 8300 3000 50  0001 C CNN
@@
 NoConn ~ 7950 2900
 $Comp
-L GND #PWR27
+L GND #PWR23
 U 1 1 5A0130C5
 P 6500 2600
-F 0 "#PWR27" H 6500 2350 50  0001 C CNN
+F 0 "#PWR23" H 6500 2350 50  0001 C CNN
 F 1 "GND" H 6500 2450 50  0000 C CNN
 F 2 "" H 6500 2600 50  0001 C CNN
@@
 	8100 2700 8100 2850
 $Comp
-L MAG3110 U4
+L MAG3110 U2
 U 1 1 5A014ADE
 P 3750 3700
-F 0 "U4" H 4150 3700 60  0000 C CNN
+F 0 "U2" H 4150 3700 60  0000 C CNN
 F 1 "MAG3110" H 3750 3700 60  0000 C CNN
 F 2 "Housings_DFN_QFN:DFN-10_2x2mm_Pitch0.4mm" H 3750 3700 60  0001 C CNN
@@
 EXT_INT_2
 $Comp
-L GND #PWR22
+L GND #PWR18
 U 1 1 5A014C7A
 P 4800 3450
-F 0 "#PWR22" H 4800 3200 50  0001 C CNN
+F 0 "#PWR18" H 4800 3200 50  0001 C CNN
 F 1 "GND" H 4800 3300 50  0000 C CNN
 F 2 "" H 4800 3450 50  0001 C CNN
@@
 SDA
 $Comp
-L +3.3V #PWR23
+L +3.3V #PWR19
 U 1 1 5A014D65
 P 5000 4050
-F 0 "#PWR23" H 5000 3900 50  0001 C CNN
+F 0 "#PWR19" H 5000 3900 50  0001 C CNN
 F 1 "+3.3V" H 5000 4190 50  0000 C CNN
 F 2 "" H 5000 4050 50  0001 C CNN
@@
 Connection ~ 5000 4050
 $Comp
-L GND #PWR24
+L GND #PWR20
 U 1 1 5A014DEF
 P 5000 4350
-F 0 "#PWR24" H 5000 4100 50  0001 C CNN
+F 0 "#PWR20" H 5000 4100 50  0001 C CNN
 F 1 "GND" H 5000 4200 50  0000 C CNN
 F 2 "" H 5000 4350 50  0001 C CNN
@@
 	4350 4050 5000 4050
 $Comp
-L GND #PWR21
+L GND #PWR17
 U 1 1 5A014E63
 P 3050 4400
-F 0 "#PWR21" H 3050 4150 50  0001 C CNN
+F 0 "#PWR17" H 3050 4150 50  0001 C CNN
 F 1 "GND" H 3050 4250 50  0000 C CNN
 F 2 "" H 3050 4400 50  0001 C CNN
@@
 	3050 4250 3050 4400
 $Comp
-L GND #PWR20
+L GND #PWR16
 U 1 1 5A014F44
 P 2700 4450
-F 0 "#PWR20" H 2700 4200 50  0001 C CNN
+F 0 "#PWR16" H 2700 4200 50  0001 C CNN
 F 1 "GND" H 2700 4300 50  0000 C CNN
 F 2 "" H 2700 4450 50  0001 C CNN
@@
 	2700 4150 3200 4150
 $Comp
-L +3.3V #PWR18
+L +3.3V #PWR14
 U 1 1 5A015071
 P 2200 3950
-F 0 "#PWR18" H 2200 3800 50  0001 C CNN
+F 0 "#PWR14" H 2200 3800 50  0001 C CNN
 F 1 "+3.3V" H 2200 4090 50  0000 C CNN
 F 2 "" H 2200 3950 50  0001 C CNN
@@
 $EndComp
 $Comp
-L GND #PWR19
+L GND #PWR15
 U 1 1 5A015106
 P 2200 4450
-F 0 "#PWR19" H 2200 4200 50  0001 C CNN
+F 0 "#PWR15" H 2200 4200 50  0001 C CNN
 F 1 "GND" H 2200 4300 50  0000 C CNN
 F 2 "" H 2200 4450 50  0001 C CNN
@@
 	2200 3950 3200 3950
 $Comp
-L GND #PWR17
+L GND #PWR13
 U 1 1 5A015490
 P 1650 4050
-F 0 "#PWR17" H 1650 3800 50  0001 C CNN
+F 0 "#PWR13" H 1650 3800 50  0001 C CNN
 F 1 "GND" H 1650 3900 50  0000 C CNN
 F 2 "" H 1650 4050 50  0001 C CNN

Commit message: Add UART level shifting.
Parts:
- renumbered C6 to C11, C7 to C12, C8 to C13, C9 to C14, C10 to C15, C11 to C16, C12 to C17, U2 to U3, U3 to U4
Changed lines of the file:
@@
 $EndDescr
 $Comp
-L LSM6DS3H U3
+L LSM6DS3H U4
 U 1 1 5A01288C
 P 7350 2650
-F 0 "U3" H 7750 2650 60  0000 C CNN
+F 0 "U4" H 7750 2650 60  0000 C CNN
 F 1 "LSM6DS3H" H 7350 2650 60  0000 C CNN
 F 2 "Housings_LGA:Bosch_LGA-14_3x2.5mm_Pitch0.5mm" H 7350 2650 60  0001 C CNN
@@
 $EndComp
 $Comp
-L GND #PWR013
+L GND #PWR29
 U 1 1 5A01298A
 P 6700 3500
-F 0 "#PWR013" H 6700 3250 50  0001 C CNN
+F 0 "#PWR29" H 6700 3250 50  0001 C CNN
 F 1 "GND" H 6700 3350 50  0000 C CNN
 F 2 "" H 6700 3500 50  0001 C CNN
@@
 Connection ~ 6700 3400
 $Comp
-L +3.3V #PWR014
+L +3.3V #PWR26
 U 1 1 5A0129F8
 P 6200 3200
-F 0 "#PWR014" H 6200 3050 50  0001 C CNN
+F 0 "#PWR26" H 6200 3050 50  0001 C CNN
 F 1 "+3.3V" H 6200 3340 50  0000 C CNN
 F 2 "" H 6200 3200 50  0001 C CNN
@@
 $EndComp
 $Comp
-L GND #PWR015
+L GND #PWR27
 U 1 1 5A012A42
 P 6200 3500
-F 0 "#PWR015" H 6200 3250 50  0001 C CNN
+F 0 "#PWR27" H 6200 3250 50  0001 C CNN
 F 1 "GND" H 6200 3350 50  0000 C CNN
 F 2 "" H 6200 3500 50  0001 C CNN
@@
 NoConn ~ 7950 3100
 $Comp
-L +3.3V #PWR016
+L +3.3V #PWR30
 U 1 1 5A012FB2
 P 8300 2700
-F 0 "#PWR016" H 8300 2550 50  0001 C CNN
+F 0 "#PWR30" H 8300 2550 50  0001 C CNN
 F 1 "+3.3V" H 8300 2840 50  0000 C CNN
 F 2 "" H 8300 2700 50  0001 C CNN
@@
 $EndComp
 $Comp
-L GND #PWR017
+L GND #PWR31
 U 1 1 5A012FF1
 P 8300 3000
-F 0 "#PWR017" H 8300 2750 50  0001 C CNN
+F 0 "#PWR31" H 8300 2750 50  0001 C CNN
 F 1 "GND" H 8300 2850 50  0000 C CNN
 F 2 "" H 8300 3000 50  0001 C CNN
@@
 NoConn ~ 7950 2900
 $Comp
-L GND #PWR018
+L GND #PWR28
 U 1 1 5A0130C5
 P 6500 2600
-F 0 "#PWR018" H 6500 2350 50  0001 C CNN
+F 0 "#PWR28" H 6500 2350 50  0001 C CNN
 F 1 "GND" H 6500 2450 50  0000 C CNN
 F 2 "" H 6500 2600 50  0001 C CNN
@@
 	8100 2700 8100 2850
 $Comp
-L MAG3110 U2
+L MAG3110 U3
 U 1 1 5A014ADE
 P 3750 3700
-F 0 "U2" H 4150 3700 60  0000 C CNN
+F 0 "U3" H 4150 3700 60  0000 C CNN
 F 1 "MAG3110" H 3750 3700 60  0000 C CNN
 F 2 "Housings_DFN_QFN:DFN-10_2x2mm_Pitch0.4mm" H 3750 3700 60  0001 C CNN
@@
 EXT_INT_2
 $Comp
-L GND #PWR019
+L GND #PWR23
 U 1 1 5A014C7A
 P 4800 3450
-F 0 "#PWR019" H 4800 3200 50  0001 C CNN
+F 0 "#PWR23" H 4800 3200 50  0001 C CNN
 F 1 "GND" H 4800 3300 50  0000 C CNN
 F 2 "" H 4800 3450 50  0001 C CNN
@@
 SDA
 $Comp
-L +3.3V #PWR020
+L +3.3V #PWR24
 U 1 1 5A014D65
 P 5000 4050
-F 0 "#PWR020" H 5000 3900 50  0001 C CNN
+F 0 "#PWR24" H 5000 3900 50  0001 C CNN
 F 1 "+3.3V" H 5000 4190 50  0000 C CNN
 F 2 "" H 5000 4050 50  0001 C CNN
@@
 Connection ~ 5000 4050
 $Comp
-L GND #PWR021
+L GND #PWR25
 U 1 1 5A014DEF
 P 5000 4350
-F 0 "#PWR021" H 5000 4100 50  0001 C CNN
+F 0 "#PWR25" H 5000 4100 50  0001 C CNN
 F 1 "GND" H 5000 4200 50  0000 C CNN
 F 2 "" H 5000 4350 50  0001 C CNN
@@
 	4350 4050 5000 4050
 $Comp
-L GND #PWR022
+L GND #PWR22
 U 1 1 5A014E63
 P 3050 4400
-F 0 "#PWR022" H 3050 4150 50  0001 C CNN
+F 0 "#PWR22" H 3050 4150 50  0001 C CNN
 F 1 "GND" H 3050 4250 50  0000 C CNN
 F 2 "" H 3050 4400 50  0001 C CNN
@@
 	3050 4250 3050 4400
 $Comp
-L GND #PWR023
+L GND #PWR21
 U 1 1 5A014F44
 P 2700 4450
-F 0 "#PWR023" H 2700 4200 50  0001 C CNN
+F 0 "#PWR21" H 2700 4200 50  0001 C CNN
 F 1 "GND" H 2700 4300 50  0000 C CNN
 F 2 "" H 2700 4450 50  0001 C CNN
@@
 	2700 4150 3200 4150
 $Comp
-L +3.3V #PWR024
+L +3.3V #PWR19
 U 1 1 5A015071
 P 2200 3950
-F 0 "#PWR024" H 2200 3800 50  0001 C CNN
+F 0 "#PWR19" H 2200 3800 50  0001 C CNN
 F 1 "+3.3V" H 2200 4090 50  0000 C CNN
 F 2 "" H 2200 3950 50  0001 C CNN
@@
 $EndComp
 $Comp
-L GND #PWR025
+L GND #PWR20
 U 1 1 5A015106
 P 2200 4450
-F 0 "#PWR025" H 2200 4200 50  0001 C CNN
+F 0 "#PWR20" H 2200 4200 50  0001 C CNN
 F 1 "GND" H 2200 4300 50  0000 C CNN
 F 2 "" H 2200 4450 50  0001 C CNN
@@
 	2200 3950 3200 3950
 $Comp
-L GND #PWR026
+L GND #PWR18
 U 1 1 5A015490
 P 1650 4050
-F 0 "#PWR026" H 1650 3800 50  0001 C CNN
+F 0 "#PWR18" H 1650 3800 50  0001 C CNN
 F 1 "GND" H 1650 3900 50  0000 C CNN
 F 2 "" H 1650 4050 50  0001 C CNN
@@
 	2900 3850 3200 3850
 $Comp
-L C C6
+L C C11
 U 1 1 5AB7EC4F
 P 1650 3900
-F 0 "C6" H 1675 4000 50  0000 L CNN
+F 0 "C11" H 1675 4000 50  0000 L CNN
 F 1 "0.1uF" H 1675 3800 50  0000 L CNN
 F 2 "Capacitors_SMD:C_1206_HandSoldering" H 1688 3750 50  0001 C CNN
@@
 $EndComp
 $Comp
-L C C8
+L C C13
 U 1 1 5AB7EE7A
 P 2300 4200
-F 0 "C8" H 2325 4300 50  0000 L CNN
+F 0 "C13" H 2325 4300 50  0000 L CNN
 F 1 "0.1uF" H 2325 4100 50  0000 L CNN
 F 2 "Capacitors_SMD:C_1206_HandSoldering" H 2338 4050 50  0001 C CNN
@@
 $EndComp
 $Comp
-L C C9
+L C C14
 U 1 1 5AB7EF1C
 P 2700 4300
-F 0 "C9" H 2725 4400 50  0000 L CNN
+F 0 "C14" H 2725 4400 50  0000 L CNN
 F 1 "0.1uF" H 2725 4200 50  0000 L CNN
 F 2 "Capacitors_SMD:C_1206_HandSoldering" H 2738 4150 50  0001 C CNN
@@
 $EndComp
 $Comp
-L C C10
+L C C15
 U 1 1 5AB7EFA4
 P 5000 4200
-F 0 "C10" H 5025 4300 50  0000 L CNN
+F 0 "C15" H 5025 4300 50  0000 L CNN
 F 1 "0.1uF" H 5025 4100 50  0000 L CNN
 F 2 "Capacitors_SMD:C_1206_HandSoldering" H 5038 4050 50  0001 C CNN
@@
 $EndComp
 $Comp
-L C C7
+L C C12
 U 1 1 5AB7F05A
 P 2050 4200
-F 0 "C7" H 2075 4300 50  0000 L CNN
+F 0 "C12" H 2075 4300 50  0000 L CNN
 F 1 "1uF" H 2075 4100 50  0000 L CNN
 F 2 "Capacitors_SMD:C_1206_HandSoldering" H 2088 4050 50  0001 C CNN
@@
 $EndComp
 $Comp
-L C C11
+L C C16
 U 1 1 5AB7F32E
 P 6200 3350
-F 0 "C11" H 6225 3450 50  0000 L CNN
+F 0 "C16" H 6225 3450 50  0000 L CNN
 F 1 "0.1uF" H 6225 3250 50  0000 L CNN
 F 2 "Housings_LGA:Bosch_LGA-14_3x2.5mm_Pitch0.5mm" H 6238 3200 50  0001 C CNN
@@
 $EndComp
 $Comp
-L C C12
+L C C17
 U 1 1 5AB7F374
 P 8300 2850
-F 0 "C12" H 8325 2950 50  0000 L CNN
+F 0 "C17" H 8325 2950 50  0000 L CNN
 F 1 "0.1uF" H 8325 2750 50  0000 L CNN
 F 2 "Capacitors_SMD:C_1206_HandSoldering" H 8338 2700 50  0001 C CNN
