File: poc_controller/poc_controller.sch (KiCad schematic (older format))
At the start: 24 parts, among them J1 CONN_01X06, J2 CONN_01X02, J3 CONN_01X02, J4 CONN_01X02, SW1 SW_DPST, U1 dsPIC33EPXXXMC502, U2 MAX232, Y1 Crystal

Commit message: WIP ECAN
Parts:
- added U?: MCP2561-E/SN, Housings_SOIC:SOIC-8_3.9x4.9mm_Pitch1.27mm, symbol MCP2561-E/SN
Changed lines of the file:
@@
 BATT_VOLT
 $Sheet
-S 9600 2150 500  150
+S 9600 2150 650  350
 U 5A10B6B3
 F0 "Motor" 60
 F1 "poc_controller_motor.sch" 60
+F2 "CAN_L" B L 9600 2250 60
+F3 "CAN_H" B L 9600 2400 60
 $EndSheet
 $Comp
@@
 Wire Wire Line
 	10600 4700 10600 4750
+$Comp
+L MCP2561-E/SN U?
+U 1 1 5ACE82D2
+P 4700 3100
+F 0 "U?" H 4300 3450 50  0000 L CNN
+F 1 "MCP2561-E/SN" H 4800 3450 50  0000 L CNN
+F 2 "Housings_SOIC:SOIC-8_3.9x4.9mm_Pitch1.27mm" H 4700 2600 50  0001 C CIN
+F 3 "" H 4700 3100 50  0001 C CNN
+	1    4700 3100
+	1    0    0    -1
+$EndComp
+Text Label 9350 2250 2    60   ~ 0
+CAN_L
+Text Label 9350 2400 2    60   ~ 0
+CAN_H
+Wire Wire Line
+	9350 2250 9600 2250
+Wire Wire Line
+	9350 2400 9600 2400
 $EndSCHEMATC
