File: poc_controller/poc_controller_motor.sch (KiCad schematic (older format))
At the start: 13 parts, among them Q1 Q_NMOS_DGS, Q2 Q_NMOS_DGS, Q3 Q_NMOS_DGS, Q4 Q_NMOS_DGS, Q5 Q_NMOS_DGS, Q6 Q_NMOS_DGS, U7 MPC8025

Commit message: More design and component selection.
Parts:
- added C16, C17, C20: 0.1uF, Capacitors_SMD:C_1206_HandSoldering, symbol C
- added C18, C19: 36pF, Capacitors_SMD:C_1206_HandSoldering, symbol C
- added C21: 10uF, Capacitors_SMD:C_1206_HandSoldering, symbol C
- added J7: CONN_01X06, Connectors:PINHEAD1-6, symbol CONN_01X06
- added R10: 4.7k, Resistors_SMD:R_1206_HandSoldering, symbol R
- added R11: 470, Resistors_SMD:R_1206_HandSoldering, symbol R
- added SW2: SW_DPST, Buttons_Switches_SMD:SW_SPST_B3SL-1022P, symbol SW_DPST
- added U6: dsPIC33EPXXXMC502, SMD_Packages:SOIC-28, symbol dsPIC33EPXXXMC502
- added Y2: Crystal, Crystals:Crystal_SMD_HC49-SD_HandSoldering, symbol Crystal
- U5: renamed from U7; footprint (none) -> Housings_QFP:TQFP-48_7x7mm_Pitch0.5mm; Part Number (none) -> 579-MCP8025-115E/PT (Mouser)
- renumbered R10 to R12, R11 to R13, R12 to R14, R13 to R15, R14 to R16, R15 to R17
Connections:
- net GND: now also C16.1, C17.2, C18.1, C19.1, C20.2, C21.2, J7.3 (P3), SW2.1, SW2.3, U6.19 (VSS), U6.8 (VSS)
- new net: C19.2, U6.10 (OSC2/CLKO/RA3), Y2.2
- new net: C21.1, U6.20 (VCAP)
- new net: C18.2, U6.9 (OSC1/CLKI/RA2), Y2.1
- new net: C17.1, R10.2, R11.2, SW2.2, SW2.4
- new net +3V3: C16.2, C20.1, J7.2 (P2), R10.1, U6.13 (VDD), U6.28 (AVDD)
- new net CPU_MCLR: J7.1 (P1), R11.1, U6.1 (MCLR)
- new net CPU_PGC: J7.5 (P5), U6.15 (PGEC2/ASCL2/RP38/RB6)
- new net CPU_PGD: J7.4 (P4), U6.14 (PGED2/ASDA2/RP37/RB5)
- no-connect marks 2 -> 3
Other:
- moved on the sheet: Q1, Q2, Q3, Q4, Q5, Q6, R12, R13, R14, R15, R16, R17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

Commit message: wip
Parts:
- added R12: 2k, Resistors_SMD:R_1206_HandSoldering, symbol R
- added R13: 22k, Resistors_SMD:R_1206_HandSoldering, symbol R
- renumbered R12 to R14, R13 to R15, R14 to R16, R15 to R17, R16 to R18, R17 to R19
Connections:
- net pwm_1_high is gone; now on net PWM_1_HIGH: U5.2 (PWM1H)
- net pwm_1_low is gone; now on net PWM_1_LOW: U5.1 (PWM1L)
- net pwm_2_high is gone; now on net PWM_2_HIGH: U5.48 (PWM2H)
- net pwm_2_low is gone; now on net PWM_2_LOW: U5.47 (PWM2L)
- net pwm_3_high is gone; now on net PWM_3_HIGH: U5.46 (PWM3H)
- net pwm_3_low is gone; now on net PWM_3_LOW: U5.45 (PWM3L)
- net +3V3: now also R13.1
- net GND: now also U5.19 (PGND), U5.20 (PGND), U5.24 (PGND), U5.35 (PGND), U5.36 (PGND), U5.4 (NC), U5.49 (EP), U5.5 (NC), U5.7 (PGND)
- net VDD: now also U5.38 (VDD), U5.39 (VDD)
- net high_side_a: no longer U5.27 (HSA)
- net high_side_b: no longer U5.26 (HSB)
- net high_side_c: no longer U5.25 (HSC)
- net low_side_a: no longer U5.21 (LSA)
- net low_side_b: no longer U5.22 (LSB)
- net low_side_c: no longer U5.23 (LSC)
- net phase_a: no longer U5.30 (PHA)
- net phase_b: no longer U5.29 (PHB)
- net phase_c: no longer U5.28 (PHC)
- net CNTRL_CE: now reaches U5.3 (CE)
- net CNTRL_CE: now also U6.5 (PGEC3/VREF+/AN3/OA1OUT/RPI33/CTED1/RB1)
- net CNTRL_RX: now reaches U5.44 (DE2)
- net CNTRL_RX: now also U6.18 (TMS/ASDA1/SDI1/RP41/RB9), R12.2
- net CNTRL_TX: now reaches U6.17 (TCK/CVREF1O/ASCL1/SDO1/RP40/T4CK/RB8)
- net CNTRL_TX: now also R12.1, R13.2
- net PWM_3_HIGH: now reaches U6.21 (TDO/RP42/PWM3H/RB10)
- net PWM_3_LOW: now reaches U6.22 (TDI/RP43/PWM3L/RB11)
- net PWM_2_HIGH: now reaches U6.23 (RPI44/PWM2H/RB12)
- net PWM_2_LOW: now reaches U6.24 (RPI45/PWM2L/CTPLS/RB13)
- net PWM_1_HIGH: now reaches U6.25 (RPI46/PWM1H/T3CK/RB14)
- net PWM_1_LOW: now reaches U6.26 (RPI47/PWM1L/T5CK/RB15)
- new net HIGH_SIDE_A: U5.27 (HSA)
- new net HIGH_SIDE_B: U5.26 (HSB)
- new net HIGH_SIDE_C: U5.25 (HSC)
- new net LOW_SIDE_A: U5.21 (LSA)
- new net LOW_SIDE_B: U5.22 (LSB)
- new net LOW_SIDE_C: U5.23 (LSC)
- new net PHASE_A_BEMF: U5.30 (PHA)
- new net PHASE_B_EMF: U5.29 (PHB)
- new net PHASE_C_BEMF: U5.28 (PHC)
- no-connect marks 3 -> 5
Other:
- moved on the sheet: C20, C21

Commit message: WIP motor controller.
Parts:
- added J?: CONN_01X03, Connectors_Terminal_Blocks:TerminalBlock_bornier-3_P5.08mm, symbol CONN_01X03
- added R?: 10k, Resistors_SMD:R_1206_HandSoldering, symbol R
- Q1, Q2, Q3, Q4, Q5, Q6: footprint (none) -> TO_SOT_Packages_SMD:TO-252-2; Part Number (none) -> FDD10AN06A0CT-ND
- R14, R15, R16, R17, R18, R19: footprint (none) -> Resistors_SMD:R_1206_HandSoldering; Part Number (none) -> 311-47ERCT-ND
Connections:
- net high_side_a is gone; now on net HIGH_SIDE_A: R14.2
- net high_side_b is gone; now on net HIGH_SIDE_B: R15.2
- net high_side_c is gone; now on net HIGH_SIDE_C: R16.2
- net low_side_a is gone; now on net LOW_SIDE_A: R19.2
- net low_side_b is gone; now on net LOW_SIDE_B: R18.2
- net low_side_c is gone; now on net LOW_SIDE_C: R17.2
- net phase_a is gone; now on net PHASE_A: Q1.1 (D), Q2.3 (S)
- net phase_b is gone; now on net PHASE_B: Q3.1 (D), Q4.3 (S)
- net phase_c is gone; now on net PHASE_C: Q5.1 (D), Q6.3 (S)
- net +3V3: now also R?.1
- net CNTRL_CE: now also U6.7 (PGED1/AN5/C1IN1-/RP35/RB3); no longer U6.5 (PGEC3/VREF+/AN3/OA1OUT/RPI33/CTED1/RB1)
- net ZC_MUX_1: now reaches U5.11 (MUX1)
- net ZC_MUX_1: now also U6.11 (FLT32/RP36/RB4)
- net ZC_MUX_2: now reaches U5.12 (MUX2)
- net ZC_MUX_2: now also U6.12 (CVREF2O/RP20/T1CK/RA4)
- net ZC_OUT: now reaches U5.13 (ZC_OUT)
- net ZC_OUT: now also U6.6 (PGEC1/AN4/C1IN1+/RPI34/RB2), R?.2
- net PHASE_A_BEMF renamed PHASE_A
- net PHASE_A: now also J?.1 (P1)
- net PHASE_B_EMF renamed PHASE_B
- net PHASE_B: now also J?.2 (P2)
- net PHASE_C_BEMF renamed PHASE_C
- net PHASE_C: now also J?.3 (P3)
- no-connect marks 5 -> 10
Other:
- moved on the sheet: C16, C18, C19, Y2

Commit message: Add UART level shifting.
Parts:
- gave numbers to parts that had none: 2
- renumbered C16 to C21, C18 to C22, C19 to C23, C17 to C24, C20 to C25, C21 to C26, J7 to J6, R12 to R13, R13 to R14, R14 to R15, R15 to R16, R16 to R17, R17 to R18, R18 to R19, R19 to R20, U5 to U6, U6 to U7
Connections:
- net CNTRL_CE: now also U7.5 (PGEC3/VREF+/AN3/OA1OUT/RPI33/CTED1/RB1); no longer U7.7 (PGED1/AN5/C1IN1-/RP35/RB3)
Changed lines of the file:
@@
 $EndComp
 $Comp
-L VDD #PWR039
+L VDD #PWR62
 U 1 1 5A14EF75
 P 8100 1250
-F 0 "#PWR039" H 8100 1100 50  0001 C CNN
+F 0 "#PWR62" H 8100 1100 50  0001 C CNN
 F 1 "VDD" H 8100 1400 50  0000 C CNN
 F 2 "" H 8100 1250 50  0001 C CNN
@@
 $EndComp
 $Comp
-L MPC8025 U5
+L MPC8025 U6
 U 1 1 5A14EFF2
 P 3900 1050
-F 0 "U5" H 4300 1050 60  0000 C CNN
+F 0 "U6" H 4300 1050 60  0000 C CNN
 F 1 "MPC8025" H 3900 1050 60  0000 C CNN
 F 2 "Housings_QFP:TQFP-48_7x7mm_Pitch0.5mm" H 3900 1050 60  0001 C CNN
@@
 Connection ~ 8300 1500
 $Comp
-L R R14
+L R R15
 U 1 1 5A14F44B
 P 7700 1850
-F 0 "R14" V 7780 1850 50  0000 C CNN
+F 0 "R15" V 7780 1850 50  0000 C CNN
 F 1 "47" V 7700 1850 50  0000 C CNN
 F 2 "Resistors_SMD:R_1206_HandSoldering" V 7630 1850 50  0001 C CNN
@@
 $EndComp
 $Comp
-L R R16
+L R R17
 U 1 1 5A14F4E4
 P 7700 2750
-F 0 "R16" V 7780 2750 50  0000 C CNN
+F 0 "R17" V 7780 2750 50  0000 C CNN
 F 1 "47" V 7700 2750 50  0000 C CNN
 F 2 "Resistors_SMD:R_1206_HandSoldering" V 7630 2750 50  0001 C CNN
@@
 	7850 1850 8000 1850
 $Comp
-L R R15
+L R R16
 U 1 1 5A14F5DB
 P 7700 2300
-F 0 "R15" V 7780 2300 50  0000 C CNN
+F 0 "R16" V 7780 2300 50  0000 C CNN
 F 1 "47" V 7700 2300 50  0000 C CNN
 F 2 "Resistors_SMD:R_1206_HandSoldering" V 7630 2300 50  0001 C CNN
@@
 Connection ~ 9450 3450
 $Comp
-L R R17
+L R R18
 U 1 1 5A14FA58
 P 7700 4050
-F 0 "R17" V 7780 4050 50  0000 C CNN
+F 0 "R18" V 7780 4050 50  0000 C CNN
 F 1 "47" V 7700 4050 50  0000 C CNN
 F 2 "Resistors_SMD:R_1206_HandSoldering" V 7630 4050 50  0001 C CNN
@@
 Connection ~ 8200 3150
 $Comp
-L R R18
+L R R19
 U 1 1 5A14FB9B
 P 7700 4650
-F 0 "R18" V 7780 4650 50  0000 C CNN
+F 0 "R19" V 7780 4650 50  0000 C CNN
 F 1 "47" V 7700 4650 50  0000 C CNN
 F 2 "Resistors_SMD:R_1206_HandSoldering" V 7630 4650 50  0001 C CNN
@@
 $EndComp
 $Comp
-L R R19
+L R R20
 U 1 1 5A14FBD8
 P 7700 5250
-F 0 "R19" V 7780 5250 50  0000 C CNN
+F 0 "R20" V 7780 5250 50  0000 C CNN
 F 1 "47" V 7700 5250 50  0000 C CNN
 F 2 "Resistors_SMD:R_1206_HandSoldering" V 7630 5250 50  0001 C CNN
@@
 LOW_SIDE_C
 $Comp
-L GND #PWR040
+L GND #PWR63
 U 1 1 5A14FEA9
 P 10200 5600
-F 0 "#PWR040" H 10200 5350 50  0001 C CNN
+F 0 "#PWR63" H 10200 5350 50  0001 C CNN
 F 1 "GND" H 10200 5450 50  0000 C CNN
 F 2 "" H 10200 5600 50  0001 C CNN
@@
 Connection ~ 9450 5450
 $Comp
-L dsPIC33EPXXXMC502 U6
+L dsPIC33EPXXXMC502 U7
 U 1 1 5AB82EBE
 P 3900 4950
-F 0 "U6" H 4600 4950 60  0000 C CNN
+F 0 "U7" H 4600 4950 60  0000 C CNN
 F 1 "dsPIC33EPXXXMC502" H 3900 4950 60  0000 C CNN
 F 2 "SMD_Packages:SOIC-28" H 3900 4950 60  0001 C CNN
@@
 $EndComp
 $Comp
-L +3.3V #PWR041
+L +3.3V #PWR58
 U 1 1 5AC176CC
 P 6400 4950
-F 0 "#PWR041" H 6400 4800 50  0001 C CNN
+F 0 "#PWR58" H 6400 4800 50  0001 C CNN
 F 1 "+3.3V" H 6400 5090 50  0000 C CNN
 F 2 "" H 6400 4950 50  0001 C CNN
@@
 $EndComp
 $Comp
-L C C20
+L C C25
 U 1 1 5AC1770A
 P 6400 5100
-F 0 "C20" H 6425 5200 50  0000 L CNN
+F 0 "C25" H 6425 5200 50  0000 L CNN
 F 1 "0.1uF" H 6425 5000 50  0000 L CNN
 F 2 "Capacitors_SMD:C_1206_HandSoldering" H 6438 4950 50  0001 C CNN
@@
 $EndComp
 $Comp
-L GND #PWR042
+L GND #PWR59
 U 1 1 5AC1775A
 P 6400 5250
-F 0 "#PWR042" H 6400 5000 50  0001 C CNN
+F 0 "#PWR59" H 6400 5000 50  0001 C CNN
 F 1 "GND" H 6400 5100 50  0000 C CNN
 F 2 "" H 6400 5250 50  0001 C CNN
@@
 Connection ~ 6400 5200
 $Comp
-L GND #PWR043
+L GND #PWR60
 U 1 1 5AC178EB
 P 6400 6000
-F 0 "#PWR043" H 6400 5750 50  0001 C CNN
+F 0 "#PWR60" H 6400 5750 50  0001 C CNN
 F 1 "GND" H 6400 5850 50  0000 C CNN
 F 2 "" H 6400 6000 50  0001 C CNN
@@
 $EndComp
 $Comp
-L GND #PWR044
+L GND #PWR44
 U 1 1 5AC179D2
 P 600 6050
-F 0 "#PWR044" H 600 5800 50  0001 C CNN
+F 0 "#PWR44" H 600 5800 50  0001 C CNN
 F 1 "GND" H 600 5900 50  0000 C CNN
 F 2 "" H 600 6050 50  0001 C CNN
@@
 $EndComp
 $Comp
-L +3.3V #PWR045
+L +3.3V #PWR45
 U 1 1 5AC17A6A
 P 600 6400
-F 0 "#PWR045" H 600 6250 50  0001 C CNN
+F 0 "#PWR45" H 600 6250 50  0001 C CNN
 F 1 "+3.3V" H 600 6540 50  0000 C CNN
 F 2 "" H 600 6400 50  0001 C CNN
@@
 $EndComp
 $Comp
-L C C16
+L C C21
 U 1 1 5AC17AAB
 P 600 6250
-F 0 "C16" H 625 6350 50  0000 L CNN
+F 0 "C21" H 625 6350 50  0000 L CNN
 F 1 "0.1uF" H 625 6150 50  0000 L CNN
 F 2 "Capacitors_SMD:C_1206_HandSoldering" H 638 6100 50  0001 C CNN
@@
 $EndComp
 $Comp
-L C C21
+L C C26
 U 1 1 5AC17E5E
 P 6600 6050
-F 0 "C21" H 6625 6150 50  0000 L CNN
+F 0 "C26" H 6625 6150 50  0000 L CNN
 F 1 "10uF" H 6625 5950 50  0000 L CNN
 F 2 "Capacitors_SMD:C_1206_HandSoldering" H 6638 5900 50  0001 C CNN
@@
 $EndComp
 $Comp
-L GND #PWR046
+L GND #PWR61
 U 1 1 5AC17EA9
 P 6600 6200
-F 0 "#PWR046" H 6600 5950 50  0001 C CNN
+F 0 "#PWR61" H 6600 5950 50  0001 C CNN
 F 1 "GND" H 6600 6050 50  0000 C CNN
 F 2 "" H 6600 6200 50  0001 C CNN
@@
 $EndComp
 $Comp
-L GND #PWR047
+L GND #PWR46
 U 1 1 5AC56463
 P 800 5050
-F 0 "#PWR047" H 800 4800 50  0001 C CNN
+F 0 "#PWR46" H 800 4800 50  0001 C CNN
 F 1 "GND" H 800 4900 50  0000 C CNN
 F 2 "" H 800 5050 50  0001 C CNN
@@
 Connection ~ 800  4750
 $Comp
-L +3.3V #PWR048
+L +3.3V #PWR49
 U 1 1 5AC56539
 P 1200 4100
-F 0 "#PWR048" H 1200 3950 50  0001 C CNN
+F 0 "#PWR49" H 1200 3950 50  0001 C CNN
 F 1 "+3.3V" H 1200 4240 50  0000 C CNN
 F 2 "" H 1200 4100 50  0001 C CNN
@@
 Connection ~ 1200 4750
 $Comp
-L C C17
+L C C24
 U 1 1 5AC56A17
 P 1200 5100
-F 0 "C17" H 1225 5200 50  0000 L CNN
+F 0 "C24" H 1225 5200 50  0000 L CNN
 F 1 "0.1uF" H 1225 5000 50  0000 L CNN
 F 2 "Capacitors_SMD:C_1206_HandSoldering" H 1238 4950 50  0001 C CNN
@@
 $EndComp
 $Comp
-L GND #PWR049
+L GND #PWR50
 U 1 1 5AC56A6D
 P 1200 5250
-F 0 "#PWR049" H 1200 5000 50  0001 C CNN
+F 0 "#PWR50" H 1200 5000 50  0001 C CNN
 F 1 "GND" H 1200 5100 50  0000 C CNN
 F 2 "" H 1200 5250 50  0001 C CNN
@@
 	1850 5100 2100 5100
 $Comp
-L CONN_01X06 J7
+L CONN_01X06 J6
 U 1 1 5AC57366
 P 1900 3500
-F 0 "J7" H 1900 3850 50  0000 C CNN
+F 0 "J6" H 1900 3850 50  0000 C CNN
 F 1 "CONN_01X06" V 2000 3500 50  0000 C CNN
 F 2 "Connectors:PINHEAD1-6" H 1900 3500 50  0001 C CNN
@@
 CPU_MCLR
 $Comp
-L +3.3V #PWR050
+L +3.3V #PWR47
 U 1 1 5AC57528
 P 1000 3250
-F 0 "#PWR050" H 1000 3100 50  0001 C CNN
+F 0 "#PWR47" H 1000 3100 50  0001 C CNN
 F 1 "+3.3V" H 1000 3390 50  0000 C CNN
 F 2 "" H 1000 3250 50  0001 C CNN
@@
 	1000 3350 1000 3250
 $Comp
-L GND #PWR051
+L GND #PWR48
 U 1 1 5AC575E5
 P 1000 3550
-F 0 "#PWR051" H 1000 3300 50  0001 C CNN
+F 0 "#PWR48" H 1000 3300 50  0001 C CNN
 F 1 "GND" H 1000 3400 50  0000 C CNN
 F 2 "" H 1000 3550 50  0001 C CNN
@@
 Connection ~ 1200 4650
 $Comp
-L C C18
+L C C22
 U 1 1 5AC58AE0
 P 950 5800
-F 0 "C18" H 975 5900 50  0000 L CNN
+F 0 "C22" H 975 5900 50  0000 L CNN
 F 1 "36pF" H 975 5700 50  0000 L CNN
 F 2 "Capacitors_SMD:C_1206_HandSoldering" H 988 5650 50  0001 C CNN
@@
 $EndComp
 $Comp
-L C C19
+L C C23
 U 1 1 5AC58B5A
 P 950 6100
-F 0 "C19" H 975 6200 50  0000 L CNN
+F 0 "C23" H 975 6200 50  0000 L CNN
 F 1 "36pF" H 975 6000 50  0000 L CNN
 F 2 "Capacitors_SMD:C_1206_HandSoldering" H 988 5950 50  0001 C CNN
@@
 PWM_1_HIGH
 $Comp
-L GND #PWR052
+L GND #PWR53
 U 1 1 5AC5A4EF
 P 2950 1850
-F 0 "#PWR052" H 2950 1600 50  0001 C CNN
+F 0 "#PWR53" H 2950 1600 50  0001 C CNN
 F 1 "GND" H 2950 1700 50  0000 C CNN
 F 2 "" H 2950 1850 50  0001 C CNN
@@
 $EndComp
 $Comp
-L GND #PWR053
+L GND #PWR52
 U 1 1 5AC5A54E
 P 2650 3600
-F 0 "#PWR053" H 2650 3350 50  0001 C CNN
+F 0 "#PWR52" H 2650 3350 50  0001 C CNN
 F 1 "GND" H 2650 3450 50  0000 C CNN
 F 2 "" H 2650 3600 50  0001 C CNN
@@
 Connection ~ 2650 3500
 $Comp
-L GND #PWR054
+L GND #PWR56
 U 1 1 5AC5A9BC
 P 5000 2400
-F 0 "#PWR054" H 5000 2150 50  0001 C CNN
+F 0 "#PWR56" H 5000 2150 50  0001 C CNN
 F 1 "GND" H 5000 2250 50  0000 C CNN
 F 2 "" H 5000 2400 50  0001 C CNN
@@
 Connection ~ 5000 2300
 $Comp
-L GND #PWR055
+L GND #PWR54
 U 1 1 5AC5AB0E
 P 4750 3700
-F 0 "#PWR055" H 4750 3450 50  0001 C CNN
+F 0 "#PWR54" H 4750 3450 50  0001 C CNN
 F 1 "GND" H 4750 3550 50  0000 C CNN
 F 2 "" H 4750 3700 50  0001 C CNN
@@
 Text Label 3350 1400 2    60   ~ 0
 CNTRL_CE
-Text Label 2100 5700 2    60   ~ 0
+Text Label 2100 5500 2    60   ~ 0
 CNTRL_CE
 $Comp
-L VDD #PWR056
+L VDD #PWR55
 U 1 1 5AC5B405
 P 4800 2650
-F 0 "#PWR056" H 4800 2500 50  0001 C CNN
+F 0 "#PWR55" H 4800 2500 50  0001 C CNN
 F 1 "VDD" H 4800 2800 50  0000 C CNN
 F 2 "" H 4800 2650 50  0001 C CNN
@@
 CNTRL_TX
 $Comp
-L R R12
+L R R13
 U 1 1 5AC5C431
 P 5300 2950
-F 0 "R12" V 5380 2950 50  0000 C CNN
+F 0 "R13" V 5380 2950 50  0000 C CNN
 F 1 "2k" V 5300 2950 50  0000 C CNN
 F 2 "Resistors_SMD:R_1206_HandSoldering" V 5230 2950 50  0001 C CNN
@@
 	5450 2950 5600 2950
 $Comp
-L +3.3V #PWR057
+L +3.3V #PWR57
 U 1 1 5AC5C6B3
 P 5500 2600
-F 0 "#PWR057" H 5500 2450 50  0001 C CNN
+F 0 "#PWR57" H 5500 2450 50  0001 C CNN
 F 1 "+3.3V" H 5500 2740 50  0000 C CNN
 F 2 "" H 5500 2600 50  0001 C CNN
@@
 $EndComp
 $Comp
-L R R13
+L R R14
 U 1 1 5AC5C715
 P 5500 2750
-F 0 "R13" V 5580 2750 50  0000 C CNN
+F 0 "R14" V 5580 2750 50  0000 C CNN
 F 1 "22k" V 5500 2750 50  0000 C CNN
 F 2 "Resistors_SMD:R_1206_HandSoldering" V 5430 2750 50  0001 C CNN
@@
 	1600 5550 800  5550
 $Comp
-L +3.3V #PWR?
+L +3.3V #PWR51
 U 1 1 5ACE1398
 P 2550 1900
-F 0 "#PWR?" H 2550 1750 50  0001 C CNN
+F 0 "#PWR51" H 2550 1750 50  0001 C CNN
 F 1 "+3.3V" H 2550 2040 50  0000 C CNN
 F 2 "" H 2550 1900 50  0001 C CNN
@@
 $EndComp
 $Comp
-L R R?
+L R R12
 U 1 1 5ACE13FD
 P 2550 2050
-F 0 "R?" V 2630 2050 50  0000 C CNN
+F 0 "R12" V 2630 2050 50  0000 C CNN
 F 1 "10k" V 2550 2050 50  0000 C CNN
 F 2 "Resistors_SMD:R_1206_HandSoldering" V 2480 2050 50  0001 C CNN
@@
 PHASE_C
 $Comp
-L CONN_01X03 J?
+L CONN_01X03 J7
 U 1 1 5ACE2FE0
 P 10650 3300
-F 0 "J?" H 10650 3500 50  0000 C CNN
+F 0 "J7" H 10650 3500 50  0000 C CNN
 F 1 "CONN_01X03" V 10750 3300 50  0000 C CNN
 F 2 "Connectors_Terminal_Blocks:TerminalBlock_bornier-3_P5.08mm" H 10650 3300 50  0001 C CNN

Commit message: WIP ECAN
Parts:
- added C?: 0.1uF, Capacitors_SMD:C_1206_HandSoldering, symbol C
- added C?: 4.7uF, Capacitors_SMD:C_1206_HandSoldering, symbol C
- added R? (x4): 120, Resistors_SMD:R_1206_HandSoldering, symbol R
- added U?: MCP2561-E/SN, Housings_SOIC:SOIC-8_3.9x4.9mm_Pitch1.27mm, symbol MCP2561-E/SN
Connections:
- net GND: now also C?.1, C?.2, U?.2 (VSS), U?.8 (STBY)
- net CAN_RX: now reaches U7.4 (PGED3/VREF-/AN2/C2IN1-/SS1/RPI32/CTED2/RB0)
- net CAN_RX: now also U?.4 (RXD)
- net CAN_TX: now reaches U7.7 (PGED1/AN5/C1IN1-/RP35/RB3)
- net CAN_TX: now also U?.1 (TXD)
- new net: C?.2, R?.1, R?.1, R?.2, R?.2, U?.5 (SPLIT)
- new net +5V: C?.1, U?.3 (VDD)
- new net CAN_H: R?.1, U?.7 (CANH)
- new net CAN_L: R?.2, U?.6 (CANL)
Changed lines of the file:
@@
 Wire Wire Line
 	10350 3400 10450 3400
+$Comp
+L MCP2561-E/SN U?
+U 1 1 5ACE8671
+P 1550 7200
+F 0 "U?" H 1150 7550 50  0000 L CNN
+F 1 "MCP2561-E/SN" H 1650 7550 50  0000 L CNN
+F 2 "Housings_SOIC:SOIC-8_3.9x4.9mm_Pitch1.27mm" H 1550 6700 50  0001 C CIN
+F 3 "" H 1550 7200 50  0001 C CNN
+F 4 "MCP2561T-E/SNCT-ND" H 1550 7200 60  0001 C CNN "Part Number"
+	1    1550 7200
+	1    0    0    -1
+$EndComp
+Text Label 2100 5400 2    60   ~ 0
+CAN_RX
+Text Label 2100 5700 2    60   ~ 0
+CAN_TX
+Text Label 1050 7000 2    60   ~ 0
+CAN_TX
+Text Label 1050 7100 2    60   ~ 0
+CAN_RX
+$Comp
+L GND #PWR?
+U 1 1 5ACE8B16
+P 1550 7600
+F 0 "#PWR?" H 1550 7350 50  0001 C CNN
+F 1 "GND" H 1550 7450 50  0000 C CNN
+F 2 "" H 1550 7600 50  0001 C CNN
+F 3 "" H 1550 7600 50  0001 C CNN
+	1    1550 7600
+	1    0    0    -1
+$EndComp
+$Comp
+L +5V #PWR?
+U 1 1 5ACE8B84
+P 3500 6800
+F 0 "#PWR?" H 3500 6650 50  0001 C CNN
+F 1 "+5V" H 3500 6940 50  0000 C CNN
+F 2 "" H 3500 6800 50  0001 C CNN
+F 3 "" H 3500 6800 50  0001 C CNN
+	1    3500 6800
+	1    0    0    -1
+$EndComp
+$Comp
+L C C?
+U 1 1 5ACE8BF2
+P 3500 6950
+F 0 "C?" H 3525 7050 50  0000 L CNN
+F 1 "0.1uF" H 3525 6850 50  0000 L CNN
+F 2 "Capacitors_SMD:C_1206_HandSoldering" H 3538 6800 50  0001 C CNN
+F 3 "" H 3500 6950 50  0001 C CNN
+F 4 "311-1179-1-ND" H 3500 6950 60  0001 C CNN "Part Number"
+	1    3500 6950
+	1    0    0    -1
+$EndComp
+$Comp
+L GND #PWR?
+U 1 1 5ACE8C83
+P 3500 7100
+F 0 "#PWR?" H 3500 6850 50  0001 C CNN
+F 1 "GND" H 3500 6950 50  0000 C CNN
+F 2 "" H 3500 7100 50  0001 C CNN
+F 3 "" H 3500 7100 50  0001 C CNN
+	1    3500 7100
+	1    0    0    -1
+$EndComp
+Wire Wire Line
+	1550 6800 1550 6650
+Wire Wire Line
+	1550 6650 3250 6650
+Wire Wire Line
+	3250 6800 3500 6800
+Connection ~ 3500 6800
+$Comp
+L C C?
+U 1 1 5ACE905A
+P 3000 7200
+F 0 "C?" H 3025 7300 50  0000 L CNN
+F 1 "4.7uF" H 3025 7100 50  0000 L CNN
+F 2 "Capacitors_SMD:C_1206_HandSoldering" H 3038 7050 50  0001 C CNN
+F 3 "" H 3000 7200 50  0001 C CNN
+F 4 "399-1230-1-ND" H 3000 7200 60  0001 C CNN "Part Number"
+	1    3000 7200
+	0    1    1    0
+$EndComp
+$Comp
+L R R?
+U 1 1 5ACE90DD
+P 2450 7350
+F 0 "R?" V 2530 7350 50  0000 C CNN
+F 1 "120" V 2450 7350 50  0000 C CNN
+F 2 "Resistors_SMD:R_1206_HandSoldering" V 2380 7350 50  0001 C CNN
+F 3 "" H 2450 7350 50  0001 C CNN
+F 4 "311-120ERCT-ND" V 2450 7350 60  0001 C CNN "Part Number"
+	1    2450 7350
+	1    0    0    -1
+$EndComp
+$Comp
+L R R?
+U 1 1 5ACE916F
+P 2450 7050
+F 0 "R?" V 2530 7050 50  0000 C CNN
+F 1 "120" V 2450 7050 50  0000 C CNN
+F 2 "Resistors_SMD:R_1206_HandSoldering" V 2380 7050 50  0001 C CNN
+F 3 "" H 2450 7050 50  0001 C CNN
+F 4 "311-120ERCT-ND" V 2450 7050 60  0001 C CNN "Part Number"
+	1    2450 7050
+	1    0    0    -1
+$EndComp
+$Comp
+L GND #PWR?
+U 1 1 5ACE93A9
+P 3150 7200
+F 0 "#PWR?" H 3150 6950 50  0001 C CNN
+F 1 "GND" H 3150 7050 50  0000 C CNN
+F 2 "" H 3150 7200 50  0001 C CNN
+F 3 "" H 3150 7200 50  0001 C CNN
+	1    3150 7200
+	0    -1   -1   0
+$EndComp
+Wire Wire Line
+	2050 7200 2850 7200
+Connection ~ 2450 7200
+Wire Wire Line
+	2050 7300 2300 7300
+Wire Wire Line
+	2300 7500 2750 7500
+Connection ~ 2450 7500
+Wire Wire Line
+	2050 7100 2300 7100
+Wire Wire Line
+	2300 7100 2300 6900
+Wire Wire Line
+	2300 6900 2800 6900
+Wire Wire Line
+	2300 7300 2300 7500
+Connection ~ 2450 6900
+Text Label 2750 7500 0    60   ~ 0
+CAN_L
+Text Label 2800 6900 0    60   ~ 0
+CAN_H
+Wire Wire Line
+	3250 6650 3250 6800
+$Comp
+L GND #PWR?
+U 1 1 5ACE9C7E
+P 950 7500
+F 0 "#PWR?" H 950 7250 50  0001 C CNN
+F 1 "GND" H 950 7350 50  0000 C CNN
+F 2 "" H 950 7500 50  0001 C CNN
+F 3 "" H 950 7500 50  0001 C CNN
+	1    950  7500
+	1    0    0    -1
+$EndComp
+Wire Wire Line
+	1050 7400 950  7400
+Wire Wire Line
+	950  7400 950  7500
+$Comp
+L R R?
+U 1 1 5ACE9E2D
+P 2650 7050
+F 0 "R?" V 2730 7050 50  0000 C CNN
+F 1 "120" V 2650 7050 50  0000 C CNN
+F 2 "Resistors_SMD:R_1206_HandSoldering" V 2580 7050 50  0001 C CNN
+F 3 "" H 2650 7050 50  0001 C CNN
+F 4 "311-120ERCT-ND" V 2650 7050 60  0001 C CNN "Part Number"
+	1    2650 7050
+	1    0    0    -1
+$EndComp
+$Comp
+L R R?
+U 1 1 5ACE9EAC
+P 2650 7350
+F 0 "R?" V 2730 7350 50  0000 C CNN
+F 1 "120" V 2650 7350 50  0000 C CNN
+F 2 "Resistors_SMD:R_1206_HandSoldering" V 2580 7350 50  0001 C CNN
+F 3 "" H 2650 7350 50  0001 C CNN
+F 4 "311-120ERCT-ND" V 2650 7350 60  0001 C CNN "Part Number"
+	1    2650 7350
+	1    0    0    -1
+$EndComp
+Connection ~ 2650 7200
+Text HLabel 1100 900  0    60   BiDi ~ 0
+CAN_H
+Text HLabel 1100 750  0    60   BiDi ~ 0
+CAN_L
+Text Label 1350 750  0    60   ~ 0
+CAN_L
+Text Label 1350 900  0    60   ~ 0
+CAN_H
+Wire Wire Line
+	1100 750  1350 750
+Wire Wire Line
+	1100 900  1350 900
 $EndSCHEMATC
